File: Controller/Controller.kicad_pcb (KiCad board)
At the start: 2 copper layers, 68.6 x 48.3 mm, 17 parts, among them J1 Barrel_Jack_CUI_PJ-102-AH, J2 Barrel_Jack_CUI_PJ-102-AH, J3 0004_4-Position-RA_43650-0412, J4 0004_4-Position-RA_43650-0412, J5 Wire_Pad_01, J6 Wire_Pad_01, M1 PCB-Module_PJRC_Teensy_3.2, M2 PCB-Module_Adafruit_096_OLED_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, SW2 Omron_B3F-1000, SW3 Omron_B3F-1000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

Commit message: Working
Parts:
- added C1: 0000100000000_100uF_UWX1C101MCL1GB, MyLib_Capacitors-SMT-Electrolytic:8mmx6.5mm, F.Cu at (96.9, 139.9)
- added D1: Lumex_SSL-LX3T453GD, MyLib_Lights-LEDs:Lumex_SSL-LX3T453GD, F.Cu at (127.4, 106.2)
- added D3: Lumex_SSL-LX3T453GD, MyLib_Lights-LEDs:Lumex_SSL-LX3T453GD, F.Cu at (116.9, 106.2)
- added D5: Lumex_SSL-LX3T453GD, MyLib_Lights-LEDs:Lumex_SSL-LX3T453GD, F.Cu at (153.9, 104.7)
- added D7: Lumex_SSL-LX3T453GD, MyLib_Lights-LEDs:Lumex_SSL-LX3T453GD, F.Cu at (141.4, 107.2)
- added J7: Wire_Pad_01, MyLib_Virtual-Board-Components:Solder_Pad_ThroughHole_45mil, F.Cu at (154.2, 125.0)
- added J8: Wire_Pad_01, MyLib_Virtual-Board-Components:Solder_Pad_ThroughHole_45mil, F.Cu at (106.6, 135.7)
- added J9: Wire_Pad_01, MyLib_Virtual-Board-Components:Solder_Pad_ThroughHole_45mil, F.Cu at (105.9, 107.2)
- added M3: No4_Screw_Mount, MyLib_Mounting_Holes:No4_Screw_Mount, F.Cu at (94.4, 105.7)
- added M4: No4_Screw_Mount, MyLib_Mounting_Holes:No4_Screw_Mount, F.Cu at (163.4, 148.7)
- added M5: No4_Screw_Mount, MyLib_Mounting_Holes:No4_Screw_Mount, F.Cu at (110.4, 144.7)
- added M6: No4_Screw_Mount, MyLib_Mounting_Holes:No4_Screw_Mount, F.Cu at (163.4, 105.7)
- added Q1: ROHM_RK7002BMT116, MyLib_Transistors-SMT:SOT-23-3, F.Cu at (109.9, 105.7)
- added R5: 00001000000_1k_MC0805WAF1001T5E-TC, MyLib_Resistors-SMT-Singles:0805, F.Cu at (149.4, 107.2)
- J1: value Barrel_Jack_CUI_PJ-102-AH -> 0002_2-Position-RA_43650-0212; footprint MyLib_Connectors-Various-Other:CUI_PJ-102-AH -> MyLib_Connectors-Molex-MicroFitJr:43650-0212; moved to B.Cu
- J2: value Barrel_Jack_CUI_PJ-102-AH -> Wire_Pad_01; footprint MyLib_Connectors-Various-Other:CUI_PJ-102-AH -> MyLib_Virtual-Board-Components:Solder_Pad_ThroughHole_45mil; moved to F.Cu
- moved J2 37.2 mm to (99.1, 113.8), turned to 0 degrees
- moved J5 10.1 mm to (102.6, 140.8)
- moved U1 7.58 mm to (134.9, 140.5)
- moved J1 7.42 mm to (101.1, 144.0)
- moved J6 6.36 mm to (94.0, 113.8)
- moved J4 3.31 mm to (122.7, 144.0)
- moved J3 3.31 mm to (147.3, 144.0)
- moved M1 0.50 mm to (94.0, 132.6)
- moved M2 0.50 mm to (157.5, 145.3)
- moved R1 0.50 mm to (110.0, 113.0)
- moved R2 0.50 mm to (122.7, 113.0)
- moved R3 0.50 mm to (135.4, 113.0)
- moved R4 0.50 mm to (148.3, 113.0)
- moved SW2 0.50 mm to (119.4, 109.7)
- moved SW3 0.50 mm to (132.1, 109.7)
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Connections:
- net Net-(M1-Pad13) renamed /MOSI
- net Net-(M1-Pad14) renamed /MISO
- net Net-(M1-Pad15) renamed /SCK
- net Net-(M1-Pad20) renamed /SDCS
- net Net-(M1-Pad21) renamed /OCS
- J1 pad 1: /SwitchPad1 -> DC_GND
- J1 pad 2: DC_GND -> +5V
- J2 pad 1: +5V -> +3.3V
- M1 pad 10: Net-(M1-Pad10) -> /LED3
- M1 pad 12: Net-(M1-Pad12) -> /Left
- M1 pad 16: /Down -> /LED7
- M1 pad 17: /Left -> /Down
- M1 pad 22: Net-(M1-Pad22) -> /LED6
- M1 pad 23: Net-(M1-Pad23) -> /LED5
- M1 pad 24: Net-(M1-Pad24) -> /RST
- M1 pad 25: Net-(M1-Pad25) -> /DC
- M1 pad 26: Net-(M1-Pad26) -> +3.3V
- M1 pad 4: Net-(M1-Pad4) -> /LED4
- M1 pad 6: Net-(M1-Pad6) -> /Button_LEDs
- M1 pad 7: Net-(M1-Pad7) -> /LED0
- M1 pad 8: Net-(M1-Pad8) -> /LED1
- M1 pad 9: Net-(M1-Pad9) -> /LED2
- M2 pad 5: Net-(M1-Pad23) -> /DC
- M2 pad 6: Net-(M1-Pad22) -> /RST
- M2 pad 9: Net-(M1-Pad26) -> +3.3V
- U1 pad 11: Net-(M1-Pad5) -> /LED7
- U1 pad 13: Net-(M1-Pad6) -> /LED6
- U1 pad 15: Net-(M1-Pad7) -> /LED5
- U1 pad 17: Net-(M1-Pad8) -> /LED4
- U1 pad 2: Net-(M1-Pad9) -> /LED0
- U1 pad 4: Net-(M1-Pad10) -> /LED1
- U1 pad 6: Net-(M1-Pad11) -> /LED2
- U1 pad 8: Net-(M1-Pad12) -> /LED3
Routing:
- net DC_GND: track 246.5 -> 42.1 mm
- net /DC: track 0.00 -> 65.1 mm
- net Net-(M1-Pad26): track 62.5 -> 0.00 mm, vias 1 -> 0
- net /RST: track 0.00 -> 61.0 mm
- net Net-(M1-Pad23): track 58.5 -> 0.00 mm
- net Net-(M1-Pad22): track 56.1 -> 0.00 mm
- net Net-(D1-Pad1): track 0.00 -> 50.6 mm
- net /LED4: track 0.00 -> 49.8 mm, vias 0 -> 1
- net /LED5: track 0.00 -> 48.1 mm, vias 0 -> 1
- net Net-(D1-Pad2): track 0.00 -> 48.0 mm
- net /LED6: track 0.00 -> 44.5 mm, vias 0 -> 1
- net Net-(M1-Pad5): track 43.1 -> 0.00 mm, vias 1 -> 0
- net Net-(M1-Pad6): track 41.2 -> 0.00 mm, vias 1 -> 0
- net /LED7: track 0.00 -> 40.6 mm, vias 0 -> 1
- net Net-(M1-Pad7): track 39.6 -> 0.00 mm, vias 1 -> 0
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- removed copper zone on F.Cu, net +5V
- removed copper zone on F.Cu, net /SwitchPad1
Other:
- board size 68.6 x 48.3 mm -> 75 x 49 mm
