File: Controller/Controller.sch (KiCad schematic (older format))
At the start: 17 parts, among them J1 Barrel_Jack_CUI_PJ-102-AH, J2 Barrel_Jack_CUI_PJ-102-AH, J3 0004_4-Position-RA_43650-0412, J4 0004_4-Position-RA_43650-0412, J5 Wire_Pad_01, J6 Wire_Pad_01, M1 PCB-Module_PJRC_Teensy_3.2, M2 PCB-Module_Adafruit_096_OLED_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, SW2 Omron_B3F-1000, SW3 Omron_B3F-1000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

Commit message: Working
Parts:
- removed J1, J2: Barrel_Jack_CUI_PJ-102-AH, MyLib_Connectors-Various-Other:CUI_PJ-102-AH, symbol Connectors_Other:Barrel_Jack_CUI_PJ-102-AH
- added C1: 0000100000000_100uF_UWX1C101MCL1GB, MyLib_Capacitors-SMT-Electrolytic:8mmx6.5mm, symbol Capacitors_Electrolytic-SMT:0000100000000_100uF_UWX1C101MCL1GB
- added D1, D3, D5, D7: Lumex_SSL-LX3T453GD, MyLib_Lights-LEDs:Lumex_SSL-LX3T453GD, symbol LEDs-Lights:Lumex_SSL-LX3T453GD
- added J1: 0002_2-Position-RA_43650-0212, MyLib_Connectors-Molex-MicroFitJr:43650-0212, symbol Connectors_MicroFitJr:0002_2-Position-RA_43650-0212
- added J2, J7, J8, J9: Wire_Pad_01, MyLib_Virtual-Board-Components:Solder_Pad_ThroughHole_45mil, symbol Connectors_Other:Wire_Pad_01
- added M3, M4, M5, M6: No4_Screw_Mount, MyLib_Mounting_Holes:No4_Screw_Mount, symbol Mounting_Holes:No4_Screw_Mount
- added Q1: ROHM_RK7002BMT116, MyLib_Transistors-SMT:SOT-23-3, symbol Transistors:ROHM_RK7002BMT116
- added R5: 00001000000_1k_MC0805WAF1001T5E-TC, MyLib_Resistors-SMT-Singles:0805, symbol Resistors_Film-SMT:00001000000_1k_MC0805WAF1001T5E-TC
Connections:
- net +5V: now also C1.1 (A), J1.2, R5.1
- net DC_GND: now also C1.2 (C), J1.1, Q1.2 (S)
- net Down: now also M1.17 (15); no longer M1.16 (14)
- net Left: now also M1.12 (10); no longer M1.17 (15)
- net at M1.5 (3): no longer U1.11 (I7)
- net Button_LEDs: now reaches M1.6 (4)
- net Button_LEDs: now also J8.1, J9.1, Q1.1 (G); no longer U1.13 (I6)
- net LED0: now reaches M1.7 (5)
- net LED0: now also U1.2 (I0); no longer U1.15 (I5)
- net LED1: now reaches M1.8 (6)
- net LED1: now also U1.4 (I1); no longer U1.17 (I4)
- net LED2: now reaches M1.9 (7)
- net LED2: now also U1.6 (I2); no longer U1.2 (I0)
- net LED3: now reaches M1.10 (8)
- net LED3: now also U1.8 (I3); no longer U1.4 (I1)
- net at M1.11 (9): no longer U1.6 (I2)
- net MOSI: now reaches M1.13 (11), M2.3 (MOSI)
- net MISO: now reaches M1.14 (12), M2.2 (MISO)
- net SCK: now reaches M1.15 (13), M2.4 (SCK)
- net SDCS: now reaches M1.20 (18), M2.8 (SDCS)
- net OCS: now reaches M1.21 (19), M2.7 (OCS)
- net LED6: now reaches M1.22 (20)
- net LED6: now also U1.13 (I6); no longer M2.6 (RST)
- net DC: now reaches M2.5 (D/C)
- net DC: now also M1.25 (23); no longer M1.23 (21)
- net RST: now reaches M1.24 (22)
- net RST: now also M2.6 (RST)
- net +3.3V: now reaches M1.26 (3.3v_out), M2.9 (VCC)
- net +3.3V: now also J2.1, J7.1
- net LED4: now reaches M1.4 (2)
- net LED4: now also U1.17 (I4)
- new net: D1.1 (C), D3.1 (C), D5.1 (C), D7.1 (C), Q1.3 (D)
- new net: D1.2 (A), D3.2 (A), D5.2 (A), D7.2 (A), R5.2
- new net LED5: M1.23 (21), U1.15 (I5)
- new net LED7: M1.16 (14), U1.11 (I7)
Other:
- moved on the sheet: J3, J4, J5, J6, M2, U1
